File: Constant_Current_PCB/last_version/hat_rpizero_tx.kicad_pcb (KiCad board)
At the start: 4 copper layers, 39.7 x 22.7 mm, 49 parts, among them Q1 2N2222AU, SW1 MK-11C04-G013, SW2 Conn_01x04, SW3 TS-1088-AR02016, U1 STM32L432KCU6, U2 MCP6001T-I/OT, U3 INA199A1DCKR, U4 TLV75533PDBVR, X1 MC-306 32.768kHz 6.0pF 20ppm

Commit message: fixed NRST
Connections:
- C9 pad 1: Net-(U1-NRST) -> NRST
- R2 pad 1: Net-(U1-NRST) -> NRST
- SW2 pad 3: /NRST -> NRST
- SW3 pad 1: Net-(U1-NRST) -> NRST
- U1 pad 4: Net-(U1-NRST) -> NRST
Routing:
- net NRST: track 0.00 -> 42.9 mm, vias 0 -> 4
- net /NRST: track 23.6 -> 0.00 mm, vias 2 -> 0
- net Net-(U1-NRST): track 18.2 -> 0.00 mm, vias 2 -> 0
